File: amplifiers/amplifiers.kicad_sch (KiCad schematic)
At the start: 0 parts

Commit message: wip save
Other:
- note added: "BJTs -- current controlled devices"
- note added: "Other Ideas: Mason Flow graphs"
Changed lines of the file:
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@@
 	(generator_version "10.0")
 	(paper "A4")
+	(rectangle
+		(start 46.736 44.196)
+		(end 153.67 83.312)
+		(stroke
+			(width 0)
+			(type dash_dot_dot)
+		)
+		(fill
+			(type none)
+		)
+	)
+	(text "Other Ideas:\nMason Flow graphs"
+		(exclude_from_sim no)
+		(at 198.12 44.196 0)
+		(effects
+			(font
+				(size 2.54 2.54)
+			)
+			(justify left)
+		)
+	)
+	(text "BJTs -- current controlled devices"
+		(exclude_from_sim no)
+		(at 81.534 41.656 0)
+		(effects
+			(font
+				(size 2.54 2.54)
+			)
+		)
+	)
 	(text "https://www.electronics-tutorials.ws/amplifier/amp_2.html"
 		(exclude_from_sim no)
