File: amplifiers/common-collector.kicad_sch (KiCad schematic)
At the start: 0 parts

Commit message: wip save
Parts:
- added C7: 3u, symbol Device:C
- added C8: 2u3, symbol Device:C
- added Q3: Q_NPN, symbol Device:Q_NPN
- added R11: 20k, symbol Device:R
- added R12: 3k6, symbol Device:R
- added R14: 220R, symbol Device:R
- added R15: 10k, symbol Device:R
- added V3: VSIN, symbol Simulation_SPICE:VSIN
Connections:
- new net: C8.2, R15.1
- new net GND: R12.2, R14.2, R15.2, V3.2
- new net VCC: Q3.C, R11.1
- new net Vin: C7.1, V3.1
- new net Vout: C8.1, Q3.E, R14.1
- new net base: C7.2, Q3.B, R11.2, R12.1
Other:
- note added: "collector is effectively "grounded" to Vcc"
- note added: "common collector amplifier (emitter/voltage follower)"
- note added: "common collector amplifier (emitter/voltage follower) * used when a high impedance input source needs to be connected to a low impedance load requiring a high current gain * output voltage tends to be unity gain and phase is in-phase"
- note added: "https://www.electronics-tutorials.ws/amplifier/common-collector-amplifier.html"

Commit message: wip save
Parts:
- added R13: 0R, symbol Device:R
- C8: value 2u3 -> 1u
- R12: value 3k6 -> 20k
- R14: value 220R -> 20k
- R15: value 10k -> 100k
Connections:
- net VCC: now also R13.1; no longer Q3.C
- new net collector: Q3.C, R13.2
Other:
- note added: "Equations: R_b = Beta (R_e + r'_e)"
- note added: "R_collector is assumed to be 0R, however in calculations, it determines if it's in active mode"
- note added: "assumptions: Vbe = 0.7v"
- note added: "common collector amplifier (emitter/voltage follower) * used when a high impedance input source needs to be connected to a low impedance load requiring a high current gain * output voltage tends to be unity gain and phase is in-phase * makes a good buffer curcuit because of near unity gain * can be used as an impedence matching curcuit * can be a good current amplifier with small changes in Ib si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"
- note added: "dc block capacitor"
- note removed: "common collector amplifier (emitter/voltage follower) * used when a high impedance input source needs to be connected to a low impedance load requiring a high current gain * output voltage tends to be unity gain and phase is in-phase"
- moved on the sheet: R12, R14, V3
