File: amplifiers/common-emitter.kicad_sch (KiCad schematic)
At the start: 10 parts, among them Q2 Q_NPN

Commit message: wip save
Other:
- note added: "common emitter amplifier (inverting amp) * output is inverted in phase * input signal source and output load share the same emitter lead of the transistor * biasing allows the transitor to prepare to receive a signal and to reduce distortion * quiescent operating point or q-point allows us to see all the possible operating points of the transistor from fully "ON" to fully "OFF" * beta value (hFE)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"
- note removed: "common emitter amplifier (inverting amp) * input signal source and output load share the same emitter lead of the transistor * biasing allows the transitor to prepare to receive a signal and to reduce distortion * quiescent operating point or q-point allows us to see all the possible operating points of the transistor from fully "ON" to fully "OFF" * beta value (hFE) is current gain"
Changed lines of the file:
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@@
 		)
 	)
-	(text "common emitter amplifier (inverting amp)\n* input signal source and output load share the same emitter lead of the transistor\n* biasing allows the transitor to prepare to receive a signal and to reduce distortion\n* quiescent operating point or q-point allows us to see all the possible operating points of the transistor from fully \"ON\" to fully \"OFF\"\n* beta value (hFE) is current gain"
+	(text "common emitter amplifier (inverting amp)\n* output is inverted in phase\n* input signal source and output load share the same emitter lead of the transistor\n* biasing allows the transitor to prepare to receive a signal and to reduce distortion\n* quiescent operating point or q-point allows us to see all the possible operating points of the transistor from fully \"ON\" to fully \"OFF\"\n* beta value (hFE) is current gain"
 		(exclude_from_sim no)
 		(at 95.758 127.508 0)
@@
 		)
 		(instances
-			(project "bjt-amp"
+			(project "amplifiers"
 				(path "/8ae523d0-1e44-401a-8c0a-127d68e06c6a/1d608d62-6b62-4129-9bf9-6774aa7c774c"
 					(reference "C4")
@@
 		)
 		(instances
-			(project "bjt-amp"
+			(project "amplifiers"
 				(path "/8ae523d0-1e44-401a-8c0a-127d68e06c6a/1d608d62-6b62-4129-9bf9-6774aa7c774c"
 					(reference "#PWR013")
@@
 		)
 		(instances
-			(project "bjt-amp"
+			(project "amplifiers"
 				(path "/8ae523d0-1e44-401a-8c0a-127d68e06c6a/1d608d62-6b62-4129-9bf9-6774aa7c774c"
 					(reference "Q2")
@@
 		)
 		(instances
-			(project "bjt-amp"
+			(project "amplifiers"
 				(path "/8ae523d0-1e44-401a-8c0a-127d68e06c6a/1d608d62-6b62-4129-9bf9-6774aa7c774c"
 					(reference "C5")
@@
 		)
 		(instances
-			(project "bjt-amp"
+			(project "amplifiers"
 				(path "/8ae523d0-1e44-401a-8c0a-127d68e06c6a/1d608d62-6b62-4129-9bf9-6774aa7c774c"
 					(reference "#PWR010")
@@
 		)
 		(instances
-			(project "bjt-amp"
+			(project "amplifiers"
 				(path "/8ae523d0-1e44-401a-8c0a-127d68e06c6a/1d608d62-6b62-4129-9bf9-6774aa7c774c"
 					(reference "R10")
@@
 		)
 		(instances
-			(project "bjt-amp"
+			(project "amplifiers"
 				(path "/8ae523d0-1e44-401a-8c0a-127d68e06c6a/1d608d62-6b62-4129-9bf9-6774aa7c774c"
 					(reference "R8")
@@
 		)
 		(instances
-			(project "bjt-amp"
+			(project "amplifiers"
 				(path "/8ae523d0-1e44-401a-8c0a-127d68e06c6a/1d608d62-6b62-4129-9bf9-6774aa7c774c"
 					(reference "R9")
@@
 		)
 		(instances
-			(project "bjt-amp"
+			(project "amplifiers"
 				(path "/8ae523d0-1e44-401a-8c0a-127d68e06c6a/1d608d62-6b62-4129-9bf9-6774aa7c774c"
 					(reference "V2")
@@
 		)
 		(instances
-			(project "bjt-amp"
+			(project "amplifiers"
 				(path "/8ae523d0-1e44-401a-8c0a-127d68e06c6a/1d608d62-6b62-4129-9bf9-6774aa7c774c"
 					(reference "C6")
@@
 		)
 		(instances
-			(project "bjt-amp"
+			(project "amplifiers"
 				(path "/8ae523d0-1e44-401a-8c0a-127d68e06c6a/1d608d62-6b62-4129-9bf9-6774aa7c774c"
 					(reference "R7")
@@
 		)
 		(instances
-			(project "bjt-amp"
+			(project "amplifiers"
 				(path "/8ae523d0-1e44-401a-8c0a-127d68e06c6a/1d608d62-6b62-4129-9bf9-6774aa7c774c"
 					(reference "#PWR08")
@@
 		)
 		(instances
-			(project "bjt-amp"
+			(project "amplifiers"
 				(path "/8ae523d0-1e44-401a-8c0a-127d68e06c6a/1d608d62-6b62-4129-9bf9-6774aa7c774c"
 					(reference "#PWR014")
@@
 		)
 		(instances
-			(project "bjt-amp"
+			(project "amplifiers"
 				(path "/8ae523d0-1e44-401a-8c0a-127d68e06c6a/1d608d62-6b62-4129-9bf9-6774aa7c774c"
 					(reference "#PWR012")
@@
 		)
 		(instances
-			(project "bjt-amp"
+			(project "amplifiers"
 				(path "/8ae523d0-1e44-401a-8c0a-127d68e06c6a/1d608d62-6b62-4129-9bf9-6774aa7c774c"
 					(reference "#PWR09")
@@
 		)
 		(instances
-			(project "bjt-amp"
+			(project "amplifiers"
 				(path "/8ae523d0-1e44-401a-8c0a-127d68e06c6a/1d608d62-6b62-4129-9bf9-6774aa7c774c"
 					(reference "#PWR011")
@@
 		)
 		(instances
-			(project "bjt-amp"
+			(project "amplifiers"
 				(path "/8ae523d0-1e44-401a-8c0a-127d68e06c6a/1d608d62-6b62-4129-9bf9-6774aa7c774c"
 					(reference "R6")

Commit message: wip save
Parts:
- added R16: 1k, symbol Device:R
Connections:
- net Vin: now also R16.1; no longer C4.1
- new net: C4.1, R16.2
Other:
- note added: "dc block capacitor"
- moved on the sheet: R10, V2
Changed lines of the file:
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@@
 	(paper "A4")
 	(rectangle
-		(start 96.012 58.42)
+		(start 106.934 58.42)
 		(end 162.306 120.396)
 		(stroke
 			(width 0)
-			(type default)
+			(type dash_dot_dot)
 		)
 		(fill
@@
 		)
 	)
+	(text "dc block\ncapacitor"
+		(exclude_from_sim no)
+		(at 150.114 68.58 0)
+		(effects
+			(font
+				(size 1.27 1.27)
+			)
+		)
+	)
 	(text "assumptions:\nb (beta) = 100\nf = 20hz"
 		(exclude_from_sim no)
-		(at 96.012 54.61 0)
+		(at 134.62 54.61 0)
 		(effects
 			(font
@@
 		)
 	)
+	(text "dc block\ncapacitor"
+		(exclude_from_sim no)
+		(at 114.554 75.184 0)
+		(effects
+			(font
+				(size 1.27 1.27)
+			)
+		)
+	)
 	(text "common emitter amplifier (inverting amp)\n* output is inverted in phase\n* input signal source and output load share the same emitter lead of the transistor\n* biasing allows the transitor to prepare to receive a signal and to reduce distortion\n* quiescent operating point or q-point allows us to see all the possible operating points of the transistor from fully \"ON\" to fully \"OFF\"\n* beta value (hFE) is current gain"
 		(exclude_from_sim no)
@@
 	(wire
 		(pts
+			(xy 102.87 87.63) (xy 110.49 87.63)
+		)
+		(stroke
+			(width 0)
+			(type default)
+		)
+	)
+	(wire
+		(pts
 			(xy 123.19 77.47) (xy 123.19 87.63)
 		)
@@
 	(wire
 		(pts
-			(xy 175.26 80.01) (xy 175.26 91.44)
+			(xy 168.91 80.01) (xy 168.91 91.44)
 		)
 		(stroke
@@
 	(wire
 		(pts
-			(xy 105.41 101.6) (xy 105.41 111.76)
+			(xy 88.9 101.6) (xy 88.9 111.76)
 		)
 		(stroke
@@
 	(wire
 		(pts
-			(xy 105.41 87.63) (xy 105.41 91.44)
-		)
-		(stroke
-			(width 0)
-			(type default)
-		)
-	)
-	(wire
-		(pts
-			(xy 153.67 80.01) (xy 175.26 80.01)
+			(xy 88.9 87.63) (xy 88.9 91.44)
+		)
+		(stroke
+			(width 0)
+			(type default)
+		)
+	)
+	(wire
+		(pts
+			(xy 153.67 80.01) (xy 168.91 80.01)
 		)
 		(stroke
@@
 	(wire
 		(pts
-			(xy 175.26 99.06) (xy 175.26 111.76)
+			(xy 168.91 99.06) (xy 168.91 111.76)
 		)
 		(stroke
@@
 	(wire
 		(pts
-			(xy 105.41 87.63) (xy 110.49 87.63)
+			(xy 88.9 87.63) (xy 95.25 87.63)
 		)
 		(stroke
@@
 	)
 	(label "Vin"
-		(at 105.41 87.63 0)
+		(at 88.9 87.63 0)
 		(effects
 			(font
@@
 			)
 			(justify left bottom)
+		)
+	)
+	(symbol
+		(lib_id "Device:R")
+		(at 99.06 87.63 90)
+		(unit 1)
+		(body_style 1)
+		(exclude_from_sim no)
+		(in_bom yes)
+		(on_board yes)
+		(in_pos_files yes)
+		(dnp no)
+		(property "Reference" "R16"
+			(at 99.06 81.28 90)
+			(show_name no)
+			(do_not_autoplace no)
+			(effects
+				(font
+					(size 1.27 1.27)
+					(thickness 0.254)
+					(bold yes)
+				)
+			)
+		)
+		(property "Value" "1k"
+			(at 99.06 83.82 90)
+			(show_name no)
+			(do_not_autoplace no)
+			(effects
+				(font
+					(size 1.27 1.27)
+					(thickness 0.254)
+					(bold yes)
+				)
+			)
+		)
+		(property "Footprint" ""
+			(at 99.06 89.408 90)
+			(hide yes)
+			(show_name no)
+			(do_not_autoplace no)
+			(effects
+				(font
+					(size 1.27 1.27)
+					(thickness 0.254)
+					(bold yes)
+				)
+			)
+		)
+		(property "Datasheet" ""
+			(at 99.06 87.63 0)
+			(hide yes)
+			(show_name no)
+			(do_not_autoplace no)
+			(effects
+				(font
+					(size 1.27 1.27)
+					(thickness 0.254)
+					(bold yes)
+				)
+			)
+		)
+		(property "Description" "Resistor"
+			(at 99.06 87.63 0)
+			(hide yes)
+			(show_name no)
+			(do_not_autoplace no)
+			(effects
+				(font
+					(size 1.27 1.27)
+					(thickness 0.254)
+					(bold yes)
+				)
+			)
+		)
+		(property "Notes" "Source"
+			(at 99.06 78.74 90)
+			(show_name no)
+			(do_not_autoplace no)
+			(effects
+				(font
+					(size 1.27 1.27)
+					(thickness 0.254)
+					(bold yes)
+				)
+			)
+		)
+		(pin "2"
+		)
+		(pin "1"
+		)
+		(instances
+			(project "amplifiers"
+				(path "/8ae523d0-1e44-401a-8c0a-127d68e06c6a/1d608d62-6b62-4129-9bf9-6774aa7c774c"
+					(reference "R16")
+					(unit 1)
+				)
+			)
 		)
 	)
@@
 	(symbol
 		(lib_id "Device:R")
-		(at 175.26 95.25 0)
+		(at 168.91 95.25 0)
 		(unit 1)
 		(body_style 1)
@@
 		(dnp no)
 		(property "Reference" "R10"
-			(at 177.8 93.9799 0)
+			(at 171.45 93.9799 0)
 			(show_name no)
 			(do_not_autoplace no)
@@
 		)
 		(property "Value" "10k"
-			(at 177.8 96.5199 0)
+			(at 171.45 96.5199 0)
 			(show_name no)
 			(do_not_autoplace no)
@@
 		)
 		(property "Footprint" ""
-			(at 173.482 95.25 90)
+			(at 167.132 95.25 90)
 			(hide yes)
 			(show_name no)
@@
 		)
 		(property "Datasheet" ""
-			(at 175.26 95.25 0)
+			(at 168.91 95.25 0)
 			(hide yes)
 			(show_name no)
@@
 		)
 		(property "Description" "Resistor"
-			(at 175.26 95.25 0)
+			(at 168.91 95.25 0)
 			(hide yes)
 			(show_name no)
@@
 		)
 		(property "Notes" "Load"
-			(at 180.086 91.186 0)
+			(at 173.736 91.186 0)
 			(show_name no)
 			(do_not_autoplace no)
@@
 	(symbol
 		(lib_id "Simulation_SPICE:VSIN")
-		(at 105.41 96.52 0)
+		(at 88.9 96.52 0)
 		(mirror y)
 		(unit 1)
@@
 		(fields_autoplaced yes)
 		(property "Reference" "V2"
-			(at 101.6 93.8501 0)
+			(at 85.09 93.8501 0)
 			(show_name no)
 			(do_not_autoplace no)
@@
 		)
 		(property "Value" "VSIN"
-			(at 101.6 96.3901 0)
+			(at 85.09 96.3901 0)
 			(show_name no)
 			(do_not_autoplace no)
@@
 		)
 		(property "Footprint" ""
-			(at 105.41 96.52 0)
+			(at 88.9 96.52 0)
 			(hide yes)
 			(show_name no)
@@
 		)
 		(property "Datasheet" "https://ngspice.sourceforge.io/docs/ngspice-html-manual/manual.xhtml#sec_Independent_Sources_for"
-			(at 105.41 96.52 0)
+			(at 88.9 96.52 0)
 			(hide yes)
 			(show_name no)
@@
 		)
 		(property "Description" "Voltage source, sinusoidal"
-			(at 105.41 96.52 0)
+			(at 88.9 96.52 0)
 			(hide yes)
 			(show_name no)
@@
 		)
 		(property "Sim.Pins" "1=+ 2=-"
-			(at 105.41 96.52 0)
+			(at 88.9 96.52 0)
 			(hide yes)
 			(show_name no)
@@
 		)
 		(property "Sim.Params" "dc=0 ampl=1 f=1k td=0 theta=0 phase=0 ac=1"
-			(at 101.6 98.9301 0)
+			(at 85.09 98.9301 0)
 			(show_name no)
 			(do_not_autoplace no)
@@
 		)
 		(property "Sim.Type" "SIN"
-			(at 105.41 96.52 0)
+			(at 88.9 96.52 0)
 			(hide yes)
 			(show_name no)
@@
 		)
 		(property "Sim.Device" "V"
-			(at 105.41 96.52 0)
+			(at 88.9 96.52 0)
 			(hide yes)
 			(show_name no)
@@
 	(symbol
 		(lib_id "power:GND")
-		(at 105.41 111.76 0)
+		(at 88.9 111.76 0)
 		(unit 1)
 		(body_style 1)
@@
 		(fields_autoplaced yes)
 		(property "Reference" "#PWR08"
-			(at 105.41 118.11 0)
+			(at 88.9 118.11 0)
 			(hide yes)
 			(show_name no)
@@
 		)
 		(property "Value" "GND"
-			(at 105.41 116.84 0)
+			(at 88.9 116.84 0)
 			(show_name no)
 			(do_not_autoplace no)
@@
 		)
 		(property "Footprint" ""
-			(at 105.41 111.76 0)
+			(at 88.9 111.76 0)
 			(hide yes)
 			(show_name no)
@@
 		)
 		(property "Datasheet" ""
-			(at 105.41 111.76 0)
+			(at 88.9 111.76 0)
 			(hide yes)
 			(show_name no)
@@
 		)
 		(property "Description" "Power symbol creates a global label with name \"GND\" , ground"
-			(at 105.41 111.76 0)
+			(at 88.9 111.76 0)
 			(hide yes)
 			(show_name no)
@@
 	(symbol
 		(lib_id "power:GND")
-		(at 175.26 111.76 0)
+		(at 168.91 111.76 0)
 		(unit 1)
 		(body_style 1)
@@
 		(fields_autoplaced yes)
 		(property "Reference" "#PWR014"
-			(at 175.26 118.11 0)
+			(at 168.91 118.11 0)
 			(hide yes)
 			(show_name no)
@@
 		)
 		(property "Value" "GND"
-			(at 175.26 116.84 0)
+			(at 168.91 116.84 0)
 			(show_name no)
 			(do_not_autoplace no)
@@
 		)
 		(property "Footprint" ""
-			(at 175.26 111.76 0)
+			(at 168.91 111.76 0)
 			(hide yes)
 			(show_name no)
@@
 		)
 		(property "Datasheet" ""
-			(at 175.26 111.76 0)
+			(at 168.91 111.76 0)
 			(hide yes)
 			(show_name no)
@@
 		)
 		(property "Description" "Power symbol creates a global label with name \"GND\" , ground"
-			(at 175.26 111.76 0)
-			(hide yes)
-			(show_name no)
+			(at 168.91 111.76 0)
+			(hide yes)
+			(show_name no)

Commit message: wip save
Parts:
- added C10: 2u3, symbol Device:C
- added C9: 3u, symbol Device:C
- added Q1: PNP, symbol Simulation_SPICE:PNP
- added R17: 100R, symbol Device:R
- added R18: 8k, symbol Device:R
- added R19: 10k, symbol Device:R
- added R20: 1k, symbol Device:R
- added R21: 900R, symbol Device:R
- added R22: 1k1, symbol Device:R
- added V4: VSIN, symbol Simulation_SPICE:VSIN
Connections:
- net GND: now also R19.2, R21.2, R22.2, V4.2
- net VCC: now also R18.1, R20.1
- net Vout: now also C10.2, R21.1
- net base: now also C9.2, Q1.2 (B), R18.2, R19.1
- net collector: now also Q1.1 (C), R22.1
- net emitter: now also C10.1, Q1.3 (E), R20.2
- net Vin: no longer names the net of R16.1, V2.1
- new net: R17.1, V4.1
- new net: C9.1, R17.2
Other:
- note added: "A_voltage = 10"
- note added: "Equations (NPN): I_base + I_collector = I_emitter β = I_collector / I_base"
- note added: "Equations (PNP): I_emitter = I_base + I_collector β = I_collector / I_base I_collector = β I_base"
- note added: "NPN"
- note added: "PNP"
- note added: "Resources: https://www.youtube.com/watch?v=ZUXG9eZfSlw&t=4s https://www.youtube.com/watch?v=g7tiBC3dCFU"
- note added: "assumptions: b (beta) = 100 f_low = 20hz V_be = 0.7v"
- note removed: "assumptions: b (beta) = 100 f = 20hz"
- moved on the sheet: C4, C5, C6, Q2, R10, R16, R6, R7, R8, R9, V2

Commit message: wip save
Other:
- note added: "Resources: https://www.youtube.com/watch?v=ZUXG9eZfSlw&t=4s https://www.youtube.com/watch?v=g7tiBC3dCFU https://www.youtube.com/watch?v=_riwtuZd-8c"
- note removed: "Resources: https://www.youtube.com/watch?v=ZUXG9eZfSlw&t=4s https://www.youtube.com/watch?v=g7tiBC3dCFU"
Changed lines of the file:
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@@
 		)
 	)
-	(text "Resources:\nhttps://www.youtube.com/watch?v=ZUXG9eZfSlw&t=4s\nhttps://www.youtube.com/watch?v=g7tiBC3dCFU"
+	(text "Resources:\nhttps://www.youtube.com/watch?v=ZUXG9eZfSlw&t=4s\nhttps://www.youtube.com/watch?v=g7tiBC3dCFU\nhttps://www.youtube.com/watch?v=_riwtuZd-8c"
 		(exclude_from_sim no)
 		(at 223.774 155.956 0)
